Commit message: keeping same naming convetions

File: ezrassor_sim_description/urdf/paver_arm.xacro (robot description, xacro)
@@ -2,508 +2,34 @@
 <robot name="ezrassor"
     xmlns:xacro="http://www.ros.org/wiki/xacro">
-    <xacro:macro name="paver_arm_link1_mesh">
+    <!-- Arm Parts -->
+    <xacro:macro name="LINK1">
         <mesh filename="file://$(find ezrassor_sim_description)/meshes/link1.dae" scale="0.35 0.35 0.35"></mesh>
     </xacro:macro>
-    <xacro:macro name="paver_arm_link2_mesh">
+    <xacro:macro name="LINK2">
         <mesh filename="file://$(find ezrassor_sim_description)/meshes/link2.dae" scale="0.35 0.35 0.35"></mesh>
     </xacro:macro>
-    <xacro:macro name="paver_arm_link3_mesh">
+    <xacro:macro name="LINK3">
         <mesh filename="file://$(find ezrassor_sim_description)/meshes/link3.dae" scale="0.35 0.35 0.35"></mesh>
     </xacro:macro>
-    <xacro:macro name="paver_arm_link4_mesh">
+    <xacro:macro name="LINK4">
         <mesh filename="file://$(find ezrassor_sim_description)/meshes/link4.dae" scale="0.35 0.35 0.35"></mesh>
     </xacro:macro>
-    <xacro:macro name="paver_arm_link5_mesh">
+    <xacro:macro name="LINK5">
         <mesh filename="file://$(find ezrassor_sim_description)/meshes/link5.dae" scale="0.35 0.35 0.35"></mesh>
     </xacro:macro>
-    <xacro:macro name="paver_arm_link6_mesh">
+    <xacro:macro name="LINK6">
         <mesh filename="file://$(find ezrassor_sim_description)/meshes/link6.dae" scale="0.35 0.35 0.45"></mesh>
     </xacro:macro>
-    <xacro:macro name="paver_arm_grabber1_mesh">
+    <xacro:macro name="GRABBER1">
         <mesh filename="file://$(find ezrassor_sim_description)/meshes/grabber1.dae" scale="0.35 0.35 0.35"></mesh>
     </xacro:macro>
-    <xacro:macro name="paver_arm_camera_mesh">
+    <xacro:macro name="CAMERA">
         <mesh filename="file://$(find ezrassor_sim_description)/meshes/arm_camera.dae" scale="0.35 0.35 0.35"></mesh>
     </xacro:macro>
-    <xacro:macro name="paver_arm_grabber2_mesh">
+    <xacro:macro name="GRABBER2">
         <mesh filename="file://$(find ezrassor_sim_description)/meshes/grabber2.dae" scale="0.35 0.35 0.35"></mesh>
     </xacro:macro>
-    <xacro:macro name="paver_arm_platform_mesh">
+    <xacro:macro name="PLATFORM">
         <mesh filename="file://$(find ezrassor_sim_description)/meshes/platform.dae" scale="2 2 2"></mesh>
     </xacro:macro>
-    <!--This xacro block sets a new paver arm for the robot.
-        Inputs:
-            arm_prefix: the name that will be used to reference this arm
-            front_facing: [true/false] represent whether or not the arm is front facing
-            link_origin: an origin tag representing the xyz,rpy for the arm link
-    -->
-    <xacro:macro name="paver_arm" params="paver_arm_prefix front_facing *link_origin">
-        <link name='link1'>
-            <pose>0 0 0 0 0 0</pose>
-            <inertial>
-            <mass value="1.0"/>
-            <origin xyz="0 0 0" rpy=" 0 0 0"/>
-            <inertia
-                ixx="0" ixy="0" ixz="0"
-                iyy="0" iyz="0"
-                izz="0"
-            />
-            </inertial>
-            <collision name='collision'>
-            <origin xyz="0 0 0" rpy=" 0 0 0"/>
-            <geometry>
-                <xacro:paver_arm_link1_mesh />
-            </geometry>
-            </collision>
-            <visual name='link1'>
-            <origin xyz="0 0 0" rpy=" 0 0 0"/>
-            <geometry>
-                <xacro:paver_arm_link1_mesh />
-            </geometry>
-            </visual>
-        </link>
-        <link name='link2'>
-            <pose>0 0 0 0 0 0</pose>
-            <inertial>
-            <mass value="1.0"/>
-            <origin xyz="0 0 0" rpy=" 0 0 0"/>
-            <inertia
-                ixx="0" ixy="0" ixz="0"
-                iyy="0" iyz="0"
-                izz="0"
-            />
-            </inertial>
-            <collision name='collision'>
-            <origin xyz="0 0.08 0.135" rpy=" 0 0 0"/>
-            <geometry>
-                <xacro:paver_arm_link2_mesh />
-            </geometry>
-            </collision>
-            <visual name='link2'>
-            <origin xyz="0 0.08 0.135" rpy=" 0 0 0"/>
-            <geometry>
-                <xacro:paver_arm_link2_mesh />
-            </geometry>
-            </visual>
-        </link>
-        <link name='link3'>
-            <pose>0 0 0 0 0 0</pose>
-            <inertial>
-            <mass value="1.0"/>
-            <origin xyz="0 0 0" rpy=" 0 0 0"/>
-            <inertia
-                ixx="0" ixy="0" ixz="0"
-                iyy="0" iyz="0"
-                izz="0"
-            />
-            </inertial>
-            <collision name='collision'>
-            <origin xyz="0.25 0.1 0" rpy=" 0 0 0"/>
-            <geometry>
-                <xacro:paver_arm_link3_mesh />
-            </geometry>
-            </collision>
-            <visual name='link3'>
-            <origin xyz="0.25 0.1 0" rpy=" 0 0 0"/>
-            <geometry>
-                <xacro:paver_arm_link3_mesh />
-            </geometry>
-            </visual>
-        </link>
-        <link name='link4'>
-            <pose>0 0 0 0 0 0</pose>
-            <inertial>
-            <mass value="1.0"/>
-            <origin xyz="0 0 0" rpy=" 0 0 0"/>
-            <inertia
-                ixx="0" ixy="0" ixz="0"
-                iyy="0" iyz="0"
-                izz="0"
-            />
-            </inertial>
-            <collision name='collision'>
-            <origin xyz="0.23 0 0" rpy=" 0 0 0"/>
-            <geometry>
-                <xacro:paver_arm_link4_mesh />
-            </geometry>
-            </collision>
-            <visual name='link4'>
-            <origin xyz="0.23 0 0" rpy=" 0 0 0"/>
-            <geometry>
-                <xacro:paver_arm_link4_mesh />
-            </geometry>
-            </visual>
-        </link>
-        <link name='link5'>
-            <pose>0 0 0 0 0 0</pose>
-            <inertial>
-            <mass value="1.0"/>
-            <origin xyz="0 0 0" rpy=" 0 0 0"/>
-            <inertia
-                ixx="0" ixy="0" ixz="0"
-                iyy="0" iyz="0"
-                izz="0"
-            />
-            </inertial>
-            <collision name='collision'>
-            <origin xyz="0 0.12 0" rpy=" 0 0 0"/>
-            <geometry>
-                <xacro:paver_arm_link5_mesh />
-            </geometry>
-            </collision>
-            <visual name='link5'>
-            <origin xyz="0 0.12 0" rpy=" 0 0 0"/>
-            <geometry>
-               <xacro:paver_arm_link5_mesh />
-            </geometry>
-            </visual>
-        </link>
-        <link name='link6'>
-            <pose>0 0 0 0 0 0</pose>
-            <inertial>
-            <mass value="1.0"/>
-            <origin xyz="0 0 0" rpy=" 0 0 0"/>
-            <inertia
-                ixx="0" ixy="0" ixz="0"
-                iyy="0" iyz="0"
-                izz="0"
-            />
-            </inertial>
-            <collision name='collision'>
-            <origin xyz="0.096 0 -0.24" rpy=" 0 0 0"/>
-            <geometry>
-                <xacro:paver_arm_link6_mesh />
-            </geometry>
-            </collision>
-            <visual name='link6'>
-            <origin xyz="0.096 0 -0.24" rpy=" 0 0 0"/>
-            <geometry>
-                 <xacro:paver_arm_link6_mesh />
-            </geometry>
-            </visual>
-        </link>
-        <link name='arm_camera'>
-            <pose>0 0 0 0 0 0</pose>
-            <inertial>
-            <mass value="0.1"/>
-            <origin xyz="0.0 0.0 0.0" rpy=" 0 0 0"/>
-            <inertia
-                ixx="0" ixy="0" ixz="0"
-                iyy="0" iyz="0"
-                izz="0"
-            />
-            </inertial>
-            <visual name='arm_camera'>
-            <origin xyz="0.04 0.0 -0.04" rpy=" 0 0 0"/>
-            <geometry>
-                <xacro:paver_arm_camera_mesh />
-            </geometry>
-            </visual>
-        </link>
-        <link name='grabber1'>
-            <pose>0 0 0 0 0 0</pose>
-            <inertial>
-            <mass value="0.1"/>
-            <origin xyz="0 0 0" rpy=" 0 0 0"/>
-            <inertia
-                ixx="0" ixy="0" ixz="0"
-                iyy="0" iyz="0"
-                izz="0"
-            />
-            </inertial>
-            <collision name='collision'>
-            <origin xyz="0 0 0" rpy=" 0 0 0"/>
-            <geometry>
-                <xacro:paver_arm_grabber1_mesh />
-            </geometry>
-            <contact_coefficients>
-                <mu>1</mu>
-            </contact_coefficients>
-            <surface>
-                <bounce>
-                <restitution_coefficient>0</restitution_coefficient>
-                </bounce>
-                <friction>
-                <ode>
-                    <fdir1>0 0 0</fdir1>
-                    <mu>1</mu>
-                    <mu2>1</mu2>
-                    <slip1>0</slip1>
-                    <slip2>0</slip2>
-                </ode>
-                </friction>
-            </surface>
-            </collision>
-            <visual name='grabber1'>
-            <origin xyz="0 0 0" rpy=" 0 0 0"/>
-            <geometry>
-                 <xacro:paver_arm_grabber1_mesh />
-            </geometry>
-            </visual>
-        </link>
-        <link name='grabber2'>
-            <pose>0 0 0 0 0 0</pose>
-            <inertial>
-            <mass value="0.1"/>
-            <origin xyz="0 0 0" rpy=" 0 0 0"/>
-            <inertia
-                ixx="0" ixy="0" ixz="0"
-                iyy="0" iyz="0"
-                izz="0"
-            />
-            </inertial>
-            <collision name='collision'>
-            <origin xyz="0 0 0" rpy=" 0 0 0"/>
-            <geometry>
-                 <xacro:paver_arm_grabber2_mesh />
-            </geometry>
-            <contact_coefficients>
-                <mu>1</mu>
-            </contact_coefficients>
-            <surface>
-                <bounce>
-                <restitution_coefficient>0</restitution_coefficient>
-                </bounce>
-                <friction>
-                <ode>
-                    <fdir1>0 0 0</fdir1>
-                    <mu>1</mu>
-                    <mu2>1</mu2>
-                    <slip1>0</slip1>
-                    <slip2>0</slip2>
-                </ode>
-                </friction>
-            </surface>
-            </collision>
-            <visual name='grabber2'>
-            <origin xyz="0 0 0" rpy=" 0 0 0"/>
-            <geometry>
-                <xacro:paver_arm_grabber2_mesh />
-            </geometry>
-            </visual>
-        </link>
-        <link name='platform'>
-            <pose>0 0 0 0 0 0</pose>
-            <inertial>
-            <mass value="1.0"/>
-            <origin xyz="0 0 0" rpy=" 0 0 0"/>
-            <inertia
-                ixx="0" ixy="0" ixz="0"
-                iyy="0" iyz="0"
-                izz="0"
-            />
-            </inertial>
-            <collision name='collision'>
-            <origin xyz="-0.5 0 0" rpy=" 0 0 0"/>
-            <geometry>
-                <box size="1 1 0.08"/>
-            </geometry>
-            <contact_coefficients>
-                <mu>1</mu>
-            </contact_coefficients>
-            </collision>
-            <visual name='platform'>
-            <origin xyz="0.1 0.06 0.1" rpy=" 0 0 0"/>
-            <geometry>
-                <xacro:paver_arm_platform_mesh />
-            </geometry>
-            </visual>
-        </link>
-        <!-- <link name="${paver_arm_prefix}">
-    		<collision name="collision">
-                <xacro:insert_block name="link_origin"/>
-    			<origin xyz="0 0 0" rpy="0 0 0"/>
-    			<geometry>
-    				<xacro:paver_arm_link1_mesh />
-    			</geometry>
-    		</collision>
-    		<visual name="visual">
-                <xacro:insert_block name="link_origin"/>
-    			<geometry>
-    				<xacro:paver_arm_link1_mesh />
-    			</geometry>
-    		</visual>
-    		<inertial>
-                <xacro:insert_block name="link_origin"/>
-    			<mass value="5"/>
-    			<xacro:cylinder_inertia m="5" r="0.05" h="0.3"/>
-    		</inertial>
-    	</link>
-        <link name="${paver_arm_prefix}">
-    		<collision name="collision">
-                <xacro:insert_block name="link_origin"/>
-    			<origin xyz="0 0 0" rpy="0 0 0"/>
-    			<geometry>
-    				<xacro:paver_arm_link2_mesh />
-    			</geometry>
-    		</collision>
-    		<visual name="visual">
-                <xacro:insert_block name="link_origin"/>
-    			<geometry>
-    				<xacro:paver_arm_link2_mesh />
-    			</geometry>
-    		</visual>
-    		<inertial>
-                <xacro:insert_block name="link_origin"/>
-    			<mass value="5"/>
-    			<xacro:cylinder_inertia m="5" r="0.05" h="0.3"/>
-    		</inertial>
-    	</link>
-        <link name="${paver_arm_prefix}">
-    		<collision name="collision">
-                <xacro:insert_block name="link_origin"/>
-    			<origin xyz="0 0 0" rpy="0 0 0"/>
-    			<geometry>
-    				<xacro:paver_arm_link3_mesh />
-    			</geometry>
-    		</collision>
-    		<visual name="visual">
-                <xacro:insert_block name="link_origin"/>
-    			<geometry>
-    				<xacro:paver_arm_link3_mesh />
-    			</geometry>
-    		</visual>
-    		<inertial>
-                <xacro:insert_block name="link_origin"/>
-    			<mass value="5"/>
-    			<xacro:cylinder_inertia m="5" r="0.05" h="0.3"/>
-    		</inertial>
-    	</link>
-        <link name="${paver_arm_prefix}">
-    		<collision name="collision">
-                <xacro:insert_block name="link_origin"/>
-    			<origin xyz="0 0 0" rpy="0 0 0"/>
-    			<geometry>
-    				<xacro:paver_arm_link4_mesh />
-    			</geometry>
-    		</collision>
-    		<visual name="visual">
-                <xacro:insert_block name="link_origin"/>
-    			<geometry>
-    				<xacro:paver_arm_link4_mesh />
-    			</geometry>
-    		</visual>
-    		<inertial>
-                <xacro:insert_block name="link_origin"/>
-    			<mass value="5"/>
-    			<xacro:cylinder_inertia m="5" r="0.05" h="0.3"/>
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