Commit message: correct models!

File: ezrassor_sim_description/urdf/ezrassor_paver_arm_rover.xacro.urdf (robot description, URDF)
Before this commit: robot ezrassor_arm, 14 links, 14 joints
Joints:
- removed joint jointRoverArmFront
- joint camera_joint: origin xyz=.3 0 -.1 rpy=0 0 0 -> xyz=0.215 0 0.05 rpy=0 0 0

File: ezrassor_sim_description/urdf/paver_arm.xacro (robot description, xacro)
@@ -19,5 +19,5 @@
     </xacro:macro>
     <xacro:macro name="LINK6">
-        <mesh filename="file://$(find ezrassor_sim_description)/meshes/link6.dae" scale="0.35 0.35 0.45"></mesh>
+        <mesh filename="file://$(find ezrassor_sim_description)/meshes/link6.1.dae" scale="0.35 0.35 0.45"></mesh>
     </xacro:macro>
     <xacro:macro name="GRABBER1">
