Commit message: Working one time autonomy movements

File: ezrassor_sim_description/urdf/ezrassor_paver_arm_rover_auto.xacro.urdf (robot description, URDF)
Before this commit: robot ezrassor_arm, 14 links, 13 joints
Links:
- link body: mass 15.0 -> 1500.0

Commit message: Adding paver models and removing frontend bugs

File: ezrassor_sim_description/urdf/ezrassor_paver_arm_rover_auto.xacro.urdf (robot description, URDF)
Before this commit: robot ezrassor_arm, 14 links, 13 joints
Links:
- link body: mass 1500.0 -> 15.0
- link grabber1: mass 0.1 -> 0.01
- link grabber2: mass 0.1 -> 0.01
- link link1: mass 1.0 -> 0.001
- link link2: mass 1.0 -> 0.001
- link link3: mass 1.0 -> 0.001
- link link4: mass 1.0 -> 0.001
- link link5: mass 1.0 -> 0.001
- link link6: mass 1.0 -> 0.001
Joints:
- joint grabber_joint1: limit lower=-0.02 upper=0.0224 effort=10 velocity=0.005 -> lower=-0.02 upper=0.0224 effort=10 velocity=0.055
- joint grabber_joint2: limit lower=-0.02 upper=0.0225 effort=10 velocity=0.005 -> lower=-0.02 upper=0.0225 effort=10 velocity=0.055
