Commit message: converting moveit config to ros2

File: ezrassor_arm_moveit_ros2/urdf/arm_model.urdf (robot description, URDF)
Before this commit: robot ezrassor, 22 links, 21 joints
Joints:
- removed joint joint0
- removed joint joint0.1
- removed joint joint1
- removed joint joint2
- removed joint joint3
- removed joint joint4
- removed joint joint5
- added joint joint12: type continuous, parent link1, child link2, origin xyz=0 -0.12 0.09 rpy=0 0 0, axis 0 0 1
- added joint joint23: type continuous, parent link2, child link3, origin xyz=0 0.037 0.13 rpy=0 0 0, axis 0 1 0
- added joint joint34: type continuous, parent link3, child link4, origin xyz=0.44 -0.037 0 rpy=0 0 0, axis 0 1 0
- added joint joint45: type continuous, parent link4, child link5, origin xyz=0.42 0.0 0 rpy=0 0 0, axis 0 1 0
- added joint joint56: type continuous, parent link5, child link6, origin xyz=0 0.12 0 rpy=0 0 0, axis 0 0 1
- added joint jointRoverLink1: type fixed, parent base_link, child link1, origin xyz=0.55 -0.1 0.27 rpy=0 0 0, axis 0 0 0

Commit message: Cleaning up autonomy

File: ezrassor_arm_moveit_ros2/urdf/arm_model.urdf (robot description, URDF)
Before this commit: robot ezrassor, 22 links, 20 joints
Joints:
- added joint joint0.1: type fixed, parent base_link, child arm_front, origin xyz=0 0 0 rpy=0 0 0, axis 0 0 0

Commit message: Loading controller on moveit

File: ezrassor_arm_moveit_ros2/urdf/arm_model.urdf (robot description, URDF)
Before this commit: robot ezrassor, 22 links, 21 joints
Joints:
- removed joint arm_back_hinge
- removed joint drum_back_hinge
- removed joint left_wheel_back_hinge
- removed joint left_wheel_front_hinge
- removed joint right_wheel_back_hinge
- removed joint right_wheel_front_hinge
- added joint arm_back_joint: type continuous, parent base_link, child arm_back, origin xyz=-0.20 0 0 rpy=0 0 0, axis 0 1 0, limit effort=100 velocity=100
- added joint drum_back_joint: type continuous, parent arm_back, child drum_back, origin xyz=-0.388245 0 0 rpy=3.1415 0 0, axis 0 1 0, limit effort=100 velocity=100
- added joint left_wheel_back_joint: type continuous, parent base_link, child left_wheel_back, origin xyz=-0.20 0.285 0 rpy=0 0 0, axis 0 1 0, limit effort=100 velocity=100
- added joint left_wheel_front_joint: type continuous, parent base_link, child left_wheel_front, origin xyz=0.20 0.285 0 rpy=0 0 0, axis 0 1 0, limit effort=100 velocity=100
- added joint right_wheel_back_joint: type continuous, parent base_link, child right_wheel_back, origin xyz=-0.20 -0.285 0 rpy=0 0 0, axis 0 1 0, limit effort=100 velocity=100
- added joint right_wheel_front_joint: type continuous, parent base_link, child right_wheel_front, origin xyz=0.20 -0.285 0 rpy=0 0 0, axis 0 1 0, limit effort=100 velocity=100
